File: DigiSynth.sch (KiCad schematic (older format))
At the start: 93 parts, among them J1 Line Out, J2 Headphone Out, J3 DIN-5, J4 Conn_01x03, J5 Conn_01x03, Q1 PZT2222A, Q2 PZT2222A, SW1 SW_Push_Dual, SW2 SW_Push_Dual, SW3 SW_Push_Dual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

Commit message: Maj #2
Parts:
- J3: symbol Connector:DIN-5 -> Connector_Generic:Conn_01x05
- J4, J5: symbol Connector:Conn_01x03 -> Connector_Generic:Conn_01x03
- Q1, Q2: symbol Transistor:BC817W -> device:Q_NPN_BEC
- U1: symbol teensy:Teensy3.2 -> DigiSynth-rescue:Teensy3.2-DigiSynth-cache
- U3: symbol opto:6N135 -> device:R_PHOTO
Connections:
- wire segments 102 -> 126
Changed lines of the file:
@@
 $EndDescr
 $Comp
-L teensy:Teensy3.2 U1
+L DigiSynth-rescue:Teensy3.2-DigiSynth-cache U1
 U 1 1 5A626E28
 P 7000 2200
@@
 	2400 3250 2550 3250
 Wire Wire Line
-	1900 2650 2100 2650
+	1900 2650 1950 2650
 Wire Wire Line
 	1950 2650 1950 2750
@@
 	1950 3250 1950 3400
 Wire Wire Line
-	1900 3250 2100 3250
+	1900 3250 1950 3250
 $Comp
 L device:C C1
@@
 	1450 2650 1600 2650
 Wire Wire Line
-	1450 2500 1450 2900
+	1450 2500 1450 2650
 Wire Wire Line
 	1450 2900 1350 2900
 Wire Wire Line
-	750  3250 1600 3250
+	750  3250 1450 3250
 Wire Wire Line
 	1450 3250 1450 3000
@@
 $EndComp
 Wire Wire Line
-	2000 1500 1450 1500
+	2000 1500 1550 1500
 Wire Wire Line
 	1450 1500 1450 1550
@@
 	1450 1550 1350 1550
 Wire Wire Line
-	1350 1650 1500 1650
+	1350 1650 1400 1650
 Wire Wire Line
 	2550 2650 2400 2650
@@
 SCK
 $Comp
-L opto:6N135 U3
+L device:R_PHOTO U3
 U 1 1 5A68FD54
 P 2400 4400
@@
 $EndComp
 $Comp
-L Connector:DIN-5 J3
+L Connector_Generic:Conn_01x05 J3
 U 1 1 5A66633D
 P 1050 4400
@@
 F 3 "http://www.mouser.com/ds/2/18/40_c091_abd_e-75918.pdf" H 1050 4400 50  0001 C CNN
 	1    1050 4400
-	1    0    0    -1
+	-1   0    0    1
 $EndComp
 $Comp
@@
 	2850 4100 2850 4200
 Wire Wire Line
-	2700 4500 3100 4500
-Wire Wire Line
 	2700 4600 2850 4600
 Wire Wire Line
@@
 Text GLabel 3100 4500 2    60   Input ~ 0
 MIDI_IN
-Connection ~ 2850 4500
 Wire Wire Line
 	1900 4300 2100 4300
@@
 $EndComp
 Wire Wire Line
-	5500 4350 5700 4350
+	5500 4350 5600 4350
 Wire Wire Line
 	5500 4550 5600 4550
 Wire Wire Line
-	5600 4250 5600 4550
+	5600 4250 5600 4350
 Connection ~ 5600 4350
 Text GLabel 5600 4250 1    60   Input ~ 0
@@
 $EndComp
 Wire Wire Line
-	7050 4350 7250 4350
+	7050 4350 7150 4350
 Wire Wire Line
 	7050 4550 7150 4550
 Wire Wire Line
-	7150 4250 7150 4550
+	7150 4250 7150 4350
 Connection ~ 7150 4350
 Text GLabel 7150 4250 1    60   Input ~ 0
@@
 $EndComp
 Wire Wire Line
-	5500 5300 5700 5300
+	5500 5300 5600 5300
 Wire Wire Line
 	5500 5500 5600 5500
 Wire Wire Line
-	5600 5200 5600 5500
+	5600 5200 5600 5300
 Connection ~ 5600 5300
 Text GLabel 5600 5200 1    60   Input ~ 0
@@
 $EndComp
 Wire Wire Line
-	7050 5300 7250 5300
+	7050 5300 7150 5300
 Wire Wire Line
 	7050 5500 7150 5500
 Wire Wire Line
-	7150 5200 7150 5500
+	7150 5200 7150 5300
 Connection ~ 7150 5300
 Text GLabel 7150 5200 1    60   Input ~ 0
@@
 $EndComp
 Wire Wire Line
-	5500 6200 5700 6200
+	5500 6200 5600 6200
 Wire Wire Line
 	5500 6400 5600 6400
 Wire Wire Line
-	5600 6100 5600 6400
+	5600 6100 5600 6200
 Connection ~ 5600 6200
 Text GLabel 5600 6100 1    60   Input ~ 0
@@
 $EndComp
 Wire Wire Line
-	5500 7050 5700 7050
+	5500 7050 5600 7050
 Wire Wire Line
 	5500 7250 5600 7250
 Wire Wire Line
-	5600 6950 5600 7250
+	5600 6950 5600 7050
 Connection ~ 5600 7050
 Text GLabel 5600 6950 1    60   Input ~ 0
@@
 $EndComp
 $Comp
-L Connector:Conn_01x03 J4
+L Connector_Generic:Conn_01x03 J4
 U 1 1 5A6F9F17
 P 550 2950
@@
 $EndComp
 $Comp
-L Connector:Conn_01x03 J5
+L Connector_Generic:Conn_01x03 J5
 U 1 1 5A6FA0D7
 P 600 1600
@@
 	2450 1050 2450 850
 $Comp
-L Transistor:BC817W Q1
+L device:Q_NPN_BEC Q1
 U 1 1 5A6658B6
 P 2550 1250
@@
 	-1   0    0    1
 $EndComp
-Connection ~ 2450 1650
 Connection ~ 2450 1500
-Wire Wire Line
-	2450 1750 2450 1450
 Wire Wire Line
 	2300 1500 2450 1500
@@
 	2900 2000 3100 2000
 Wire Wire Line
-	3100 1950 3100 2050
-$Comp
-L Transistor:BC817W Q2
+	3100 1950 3100 2000
+$Comp
+L device:Q_NPN_BEC Q2
 U 1 1 5A6A3042
 P 3200 1750
@@
 	3400 1750 3400 1450
 Wire Wire Line
-	3250 1450 4100 1450
-Wire Wire Line
-	3250 1150 3250 1450
-Wire Wire Line
-	2750 1250 3400 1250
+	3250 1450 3400 1450
+Wire Wire Line
+	3250 1150 3250 1250
+Wire Wire Line
+	2750 1250 3250 1250
 Connection ~ 3250 1250
 $Comp
@@
 Text GLabel 1200 5850 0    60   Input ~ 0
 SS
+Wire Wire Line
+	1950 2650 2100 2650
+Wire Wire Line
+	1950 3250 2100 3250
+Wire Wire Line
+	5600 4350 5700 4350
+Wire Wire Line
+	5600 4350 5600 4550
+Wire Wire Line
+	7150 4350 7250 4350
+Wire Wire Line
+	7150 4350 7150 4550
+Wire Wire Line
+	5600 5300 5700 5300
+Wire Wire Line
+	5600 5300 5600 5500
+Wire Wire Line
+	7150 5300 7250 5300
+Wire Wire Line
+	7150 5300 7150 5500
+Wire Wire Line
+	5600 6200 5700 6200
+Wire Wire Line
+	5600 6200 5600 6400
+Wire Wire Line
+	5600 7050 5700 7050
+Wire Wire Line
+	5600 7050 5600 7250
+Wire Wire Line
+	1550 1500 1450 1500
+Wire Wire Line
+	1400 1650 1500 1650
+Wire Wire Line
+	1450 2650 1450 2900
+Wire Wire Line
+	1450 3250 1600 3250
+Wire Wire Line
+	2450 1500 2450 1450
+Wire Wire Line
+	3100 2000 3100 2050
+Wire Wire Line
+	3250 1250 3250 1450
+Wire Wire Line
+	3250 1250 3400 1250
+Wire Wire Line
+	3400 1450 3650 1450
+Wire Wire Line
+	3650 1450 4100 1450
+Wire Wire Line
+	2700 4500 3100 4500
+Wire Wire Line
+	2450 1500 2450 1750
 $EndSCHEMATC
